Commit message: Steering Adjusted

File: Limo_robot_dev_mk2/src/limo_ros2/limo_car/gazebo/ackermann.xacro (robot description, xacro)
@@ -79,6 +79,6 @@
             <axis xyz="0 0 1" />
             <!-- Paramenten von Herstellern -->
-            <limit lower="-0.523598767" upper="0.523598767" effort="5" velocity="0.5" />
-            <dynamics damping="1.0" friction="2.0"/>
+            <limit lower="-0.523598767" upper="0.523598767" effort="20" velocity="3.0" />
+            <dynamics damping="0.1" friction="0.1"/>
         </joint>
         <transmission name="${wheel_prefix}_hinge_trans" type="SimpleTransmission">
@@ -151,6 +151,6 @@
             <xacro:insert_block name="joint_pose"/>
             <axis xyz="0 0 -1"/>
-            <limit lower="-0.523598767" upper="0.523598767" effort="5" velocity="0.5" />
-            <dynamics damping="1.0" friction="2.0"/>
+            <limit lower="-0.523598767" upper="0.523598767" effort="20" velocity="3.0" />
+            <dynamics damping="0.1" friction="0.1"/>
         </joint>
         <transmission name="${wheel_prefix}_hinge_trans" type="SimpleTransmission">
