Commit message: Resolution and camera perfected

File: Limo_robot_dev_mk2/src/limo_ros2/limo_car/gazebo/ackermann_with_sensor.xacro (robot description, xacro)
@@ -20,5 +20,5 @@
     <xacro:gazebo_depth_camera frame_prefix="depth_camera" />
     <joint name="depth_camera_joint" type="fixed">
-        <origin xyz="0.1 0 0.065" rpy="0 0 0"/>
+        <origin xyz="0.1 0 0.065" rpy="0 0.35 0"/>
         <parent link="base_link"/>
         <child link="depth_camera_link"/>

File: Limo_robot_dev_mk2/src/limo_ros2/limo_car/gazebo/sensor.xacro (robot description, xacro)
@@ -121,5 +121,5 @@
                 <update_rate>20.0</update_rate>
                 <camera name="head">
-                    <horizontal_fov>1.3962634</horizontal_fov> <!-- 60*pi/180 -->
+                    <horizontal_fov>1.0471976</horizontal_fov> <!-- 60*pi/180 -->
                     <!-- normalisieren die Form für Fotos -->
                     <image>

Commit message: Base_CV completed

File: Limo_robot_dev_mk2/src/limo_ros2/limo_car/gazebo/ackermann_with_sensor.xacro (robot description, xacro)
@@ -20,5 +20,5 @@
     <xacro:gazebo_depth_camera frame_prefix="depth_camera" />
     <joint name="depth_camera_joint" type="fixed">
-        <origin xyz="0.1 0 0.065" rpy="0 0.35 0"/>
+        <origin xyz="0.1 0 0.065" rpy="0 0 0"/>
         <parent link="base_link"/>
         <child link="depth_camera_link"/>
